File: investigations/RFPowerAmp/FDT86256.kicad_sch (KiCad schematic)
At the start: 17 parts, among them J401 5-1814832-1, J402 5-1814832-1, Q401 FDT86246

Commit message: Re-organizing source code
Parts:
- C? (x2): PartNo (none) -> C0805C102K5RAC7800
- C? (x3): PartNo (none) -> C0805C104K1RAC7800
Changed lines of the file:
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@@
+      (effects (font (size 1.27 1.27)) hide)
+    )
+    (property "PartNo" "C0805C102K5RAC7800" (at 58.42 40.64 0)
       (effects (font (size 1.27 1.27)) hide)
     )
@@
       (effects (font (size 1.27 1.27)) hide)
     )
+    (property "PartNo" "C0805C104K1RAC7800" (at 77.47 40.64 0)
+      (effects (font (size 1.27 1.27)) hide)
+    )
     (pin "1")
     (pin "2")
@@
     )
     (property "Datasheet" "~" (at 130.81 55.88 0)
+      (effects (font (size 1.27 1.27)) hide)
+    )
+    (property "PartNo" "C0805C104K1RAC7800" (at 130.81 55.88 90)
       (effects (font (size 1.27 1.27)) hide)
     )
@@
     )
     (property "Datasheet" "~" (at 96.52 40.64 0)
+      (effects (font (size 1.27 1.27)) hide)
+    )
+    (property "PartNo" "C0805C104K1RAC7800" (at 96.52 40.64 0)
       (effects (font (size 1.27 1.27)) hide)
     )
@@
       (effects (font (size 1.27 1.27)) hide)
     )
+    (property "PartNo" "C0805C102K5RAC7800" (at 110.49 40.64 0)
+      (effects (font (size 1.27 1.27)) hide)
+    )
