File: investigations/RFPowerAmp/IRF510.kicad_sch (KiCad schematic)
At the start: 17 parts, among them J201 5-1814832-1, J202 5-1814832-1

Commit message: Re-organizing source code
Parts:
- C? (x2): PartNo (none) -> C0805C102K5RAC7800
- C? (x2): PartNo (none) -> C0805C104K1RAC7800
- C?: value 100 nF, 100 V -> 100 nF; PartNo (none) -> C0805C104K1RAC7800
Changed lines of the file:
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@@
       (effects (font (size 1.27 1.27)) hide)
     )
-    (property "Datasheet" "~" (at 64.77 60.96 0)
+    (property "Datasheet" "https://www.digikey.com/en/products/detail/kemet/C0805C102K5RAC7800/411146" (at 64.77 60.96 0)
+      (effects (font (size 1.27 1.27)) hide)
+    )
+    (property "PartNo" "C0805C102K5RAC7800" (at 64.77 60.96 0)
       (effects (font (size 1.27 1.27)) hide)
     )
@@
       (effects (font (size 1.27 1.27)) hide)
     )
+    (property "PartNo" "C0805C104K1RAC7800" (at 102.87 60.96 0)
+      (effects (font (size 1.27 1.27)) hide)
+    )
     (pin "1")
     (pin "2")
@@
       (effects (font (size 1.27 1.27)))
     )
-    (property "Value" "100 nF, 100 V" (at 137.16 71.12 90)
+    (property "Value" "100 nF" (at 137.16 71.12 90)
       (effects (font (size 1.27 1.27)))
     )
@@
     )
     (property "Datasheet" "~" (at 137.16 76.2 0)
+      (effects (font (size 1.27 1.27)) hide)
+    )
+    (property "PartNo" "C0805C104K1RAC7800" (at 137.16 76.2 90)
       (effects (font (size 1.27 1.27)) hide)
     )
@@
     )
     (property "Datasheet" "~" (at 83.82 60.96 0)
+      (effects (font (size 1.27 1.27)) hide)
+    )
+    (property "PartNo" "C0805C104K1RAC7800" (at 83.82 60.96 0)
       (effects (font (size 1.27 1.27)) hide)
     )
@@
       (effects (font (size 1.27 1.27)) hide)
     )
+    (property "PartNo" "C0805C102K5RAC7800" (at 116.84 60.96 0)
+      (effects (font (size 1.27 1.27)) hide)
+    )
