File: investigations/RFPowerAmp/FDC8602.kicad_sch (KiCad schematic)
At the start: 24 parts, among them J401 5-1814832-1, J402 5-1814832-1, J504 CONN_20, J505 CONN_20, Q501 FDC8602, T501 BN-43-202, U1 L7805CV, U501 74ACT86

Commit message: Re-organizing source code
Parts:
- C102: PartNo (none) -> C0805C224K1RAC7800
- C103, C? (x3): PartNo (none) -> C0805C104K1RAC7800
- C? (x3): PartNo (none) -> C0805C102K5RAC7800
Changed lines of the file:
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@@
+      (effects (font (size 1.27 1.27)) hide)
+    )
+    (property "PartNo" "C0805C224K1RAC7800" (at 138.43 130.81 0)
       (effects (font (size 1.27 1.27)) hide)
     )
@@
       (effects (font (size 1.27 1.27)) hide)
     )
+    (property "PartNo" "C0805C104K1RAC7800" (at 113.03 66.04 0)
+      (effects (font (size 1.27 1.27)) hide)
+    )
     (pin "1")
     (pin "2")
@@
     )
     (property "Datasheet" "~" (at 90.17 44.45 0)
+      (effects (font (size 1.27 1.27)) hide)
+    )
+    (property "PartNo" "C0805C102K5RAC7800" (at 90.17 44.45 0)
       (effects (font (size 1.27 1.27)) hide)
     )
@@
       (effects (font (size 1.27 1.27)) hide)
     )
+    (property "PartNo" "C0805C102K5RAC7800" (at 127 66.04 0)
+      (effects (font (size 1.27 1.27)) hide)
+    )
     (pin "1")
     (pin "2")
@@
       (effects (font (size 1.27 1.27)) hide)
     )
+    (property "PartNo" "C0805C104K1RAC7800" (at 175.26 62.23 0)
+      (effects (font (size 1.27 1.27)) hide)
+    )
     (pin "1")
     (pin "2")
@@
     )
     (property "Datasheet" "~" (at 154.94 50.8 0)
+      (effects (font (size 1.27 1.27)) hide)
+    )
+    (property "PartNo" "C0805C102K5RAC7800" (at 154.94 50.8 90)
       (effects (font (size 1.27 1.27)) hide)
     )
@@
       (effects (font (size 1.27 1.27)) hide)
     )
+    (property "PartNo" "C0805C104K1RAC7800" (at 102.87 44.45 0)
+      (effects (font (size 1.27 1.27)) hide)
+    )
     (pin "1")
     (pin "2")
@@
       (effects (font (size 1.27 1.27)) hide)
     )
+    (property "PartNo" "C0805C104K1RAC7800" (at 107.95 130.81 0)
+      (effects (font (size 1.27 1.27)) hide)
+    )

Commit message: Moving Pwr/tcxo to its own sheet
Parts:
- removed C101: 10 uF, Capacitors:PANASONIC_C, symbol Device:C_Polarized
- removed C102: 220 nF, Capacitor_SMD:C_0805_2012Metric, symbol Device:C
- removed C103: 100 nF, symbol Device:C
- removed J505: CONN_20, 1X20, symbol SparkFun-Connectors:CONN_20
- removed U1: L7805CV, digikey-footprints:TO-220-3, symbol dk_PMIC-Voltage-Regulators-Linear:L7805CV
- J401: value 5-1814832-1 -> Clk In
- J401: value 5-1814832-1 -> Key Shape In
- J402: value 5-1814832-1 -> RF Out
- TP?: value Output -> RF Out
- TP?: value Keyed -> Vdd
Connections:
- no-connect marks 34 -> 14

Commit message: Updates .gitignore and investigations
Connections:
- net GND: no longer J504.3
- net at J401.2, U501.1, U501.10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: no longer J504.2
- no-connect marks 14 -> 16
Changed lines of the file:
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@@
   (junction (at 83.82 40.64) (diameter 0) (color 0 0 0 0)
   )
-  (junction (at 78.74 114.3) (diameter 0) (color 0 0 0 0)
-  )
   (junction (at 78.74 81.28) (diameter 0) (color 0 0 0 0)
   )
@@
   )
   (junction (at 83.82 109.22) (diameter 0) (color 0 0 0 0)
-  )
-  (junction (at 66.04 119.38) (diameter 0) (color 0 0 0 0)
   )
   (junction (at 78.74 90.17) (diameter 0) (color 0 0 0 0)
@@
   (no_connect (at 63.5 129.54))
   (no_connect (at 63.5 149.86))
+  (no_connect (at 63.5 119.38))
   (no_connect (at 63.5 160.02))
   (no_connect (at 63.5 154.94))
   (no_connect (at 63.5 134.62))
   (no_connect (at 63.5 139.7))
+  (no_connect (at 63.5 116.84))
   (wire (pts (xy 151.13 50.8) (xy 146.05 50.8))
     (stroke (width 0) (type default))
@@
     (stroke (width 0) (type default))
   )
-  (wire (pts (xy 63.5 119.38) (xy 66.04 119.38))
-    (stroke (width 0) (type default))
-  )
   (wire (pts (xy 129.54 46.99) (xy 129.54 43.18))
     (stroke (width 0) (type default))
@@
     (stroke (width 0) (type default))
   )
-  (wire (pts (xy 66.04 119.38) (xy 66.04 114.3))
-    (stroke (width 0) (type default))
-  )
   (wire (pts (xy 86.36 114.3) (xy 78.74 114.3))
     (stroke (width 0) (type default))
   )
-  (wire (pts (xy 78.74 116.84) (xy 78.74 114.3))
-    (stroke (width 0) (type default))
-  )
   (wire (pts (xy 86.36 86.36) (xy 83.82 86.36))
     (stroke (width 0) (type default))
   )
-  (wire (pts (xy 63.5 116.84) (xy 78.74 116.84))
-    (stroke (width 0) (type default))
-  )
   (wire (pts (xy 83.82 72.39) (xy 83.82 40.64))
     (stroke (width 0) (type default))
@@
     (stroke (width 0) (type default))
   )
-  (wire (pts (xy 66.04 119.38) (xy 66.04 162.56))
+  (wire (pts (xy 66.04 114.3) (xy 66.04 162.56))
     (stroke (width 0) (type default))
   )
@@
     (stroke (width 0) (type default))
   )
-  (text_box "Pins\n 1 - Ground\n 2 - Clk In\n 3 - Ground\n 5 - +5V\n12 - +12V\n19 - Alignment Plug\n20 - Ground"
+  (text_box "Pins\n 1 - Ground\n 3 - +3V\n 5 - +5V\n12 - +12V\n19 - Alignment Plug\n20 - Ground"
     (at 73.66 149.86 0) (size 25.4 27.94)
     (stroke (width 0) (type default))

Commit message: simulations
Parts:
- gave numbers to parts that had none: 10
- renumbered J401 to J501, J401 to J502, J402 to J503, R201 to R502, R201 to R503
